File: PCB.sch (KiCad schematic (older format))
At the start: 23 parts, among them J1 Power_Connectors

Commit message: finished pcb layout
Parts:
- C3: footprint Capacitor_THT:CP_Radial_D4.0mm_P1.50mm -> Capacitor_THT:CP_Radial_D4.0mm_P2.00mm
- J2: renamed from J?; DIgiKey CP-102AH-ND -> (none); DigiKey (none) -> CP-102AH-ND
- R1, R2, R3, R4: footprint Resistor_THT:R_Axial_DIN0411_L9.9mm_D3.6mm_P15.24mm_Horizontal -> Resistor_THT:R_Axial_DIN0207_L6.3mm_D2.5mm_P7.62mm_Horizontal
- renumbered L7809CV to L7809CV1, LF33CV to LF33CV1, LM7805ACT to LM7805ACT1
Other:
- moved on the sheet: D1, D2, D3, D4, R1, R2, R3, R4
